Commit message: fwmax urdf color change

File: urdf/fwmax_skid_steer.urdf.xacro (robot description, xacro)
@@ -8,4 +8,6 @@
   <xacro:property name="wheel_radius" value="0.125"/>
   <xacro:property name="wheel_width" value="0.080"/>
+  <xacro:property name="wheel_visual_radius" value="0.128"/>
+  <xacro:property name="wheel_visual_width" value="0.105"/>
   <xacro:property name="wheelbase" value="0.600"/>
   <xacro:property name="wheel_track" value="0.450"/>
@@ -20,6 +22,9 @@
   <xacro:property name="base_com_z" value="0.008694214876"/>
   <xacro:property name="wheel_mass" value="1.0"/>
+  <material name="fwmax_body_dark_silver">
+    <color rgba="0.32 0.34 0.37 1.0"/>
+  </material>
   <material name="fwmax_wheel_black">
-    <color rgba="0.08 0.08 0.08 1.0"/>
+    <color rgba="0.02 0.02 0.025 1.0"/>
   </material>
   <!-- Keep the inertial base_link below a massless KDL-compatible root. -->
@@ -41,4 +46,5 @@
           scale="1 1 1"/>
       </geometry>
+      <material name="fwmax_body_dark_silver"/>
     </visual>
     <!-- Keep the expensive detailed DAE out of the contact calculation. -->
@@ -72,5 +78,6 @@
         <origin xyz="0 0 0" rpy="1.57079632679 0 0"/>
         <geometry>
-          <cylinder radius="0.120" length="0.060"/>
+          <cylinder
+            radius="${wheel_visual_radius}" length="${wheel_visual_width}"/>
         </geometry>
         <material name="fwmax_wheel_black"/>

Commit message: add prismatic joint on fwmax wheels as suspension

File: urdf/fwmax_skid_steer.urdf.xacro (robot description, xacro)
@@ -14,11 +14,20 @@
   <xacro:property name="base_height" value="0.388"/>
   <xacro:property name="wheel_center_z" value="${wheel_radius - base_height}"/>
+  <!-- Positive joint travel compresses the wheel upward toward the chassis. -->
+  <xacro:property name="suspension_lower_limit" value="-0.030"/>
+  <xacro:property name="suspension_upper_limit" value="0.040"/>
+  <xacro:property name="suspension_stiffness" value="20000.0"/>
+  <xacro:property name="suspension_damping" value="925.0"/>
+  <!-- Preload supports the 117 kg sprung chassis at zero joint travel. -->
+  <xacro:property name="suspension_reference" value="-0.0143471"/>
   <!--
-    Total mass is 125 kg: 121 kg for the chassis and 1 kg per wheel.
-    The chassis inertial offset compensates for the four wheel masses so the
-    assembled robot's centre of mass is at the base_link origin.
+    Total mass is 125 kg: 117 kg for the chassis, plus a 1 kg suspension
+    carrier and a 1 kg wheel at each corner. The chassis inertial offset makes
+    the assembled robot's centre of mass coincide with the base_link origin at
+    the designed loaded equilibrium position (zero joint travel).
   -->
-  <xacro:property name="base_mass" value="121.0"/>
-  <xacro:property name="base_com_z" value="0.008694214876"/>
+  <xacro:property name="base_mass" value="117.0"/>
+  <xacro:property name="base_com_z" value="0.017982905983"/>
+  <xacro:property name="suspension_mass" value="1.0"/>
   <xacro:property name="wheel_mass" value="1.0"/>
   <material name="fwmax_body_dark_silver">
@@ -36,6 +45,6 @@
       <!-- Box approximation based on the 0.96 x 0.55 x 0.395 m envelope. -->
       <inertia
-        ixx="4.623460417" ixy="0.0" ixz="0.0"
-        iyy="10.866052083" iyz="0.0" izz="12.343008333"/>
+        ixx="4.470618750" ixy="0.0" ixz="0.0"
+        iyy="10.506843750" iyz="0.0" izz="11.934975000"/>
     </inertial>
     <visual name="fwmax_dae_visual">
@@ -62,4 +71,30 @@
   </joint>
   <xacro:macro name="fwmax_wheel" params="prefix x y">
+    <link name="${prefix}_suspension_link">
+      <inertial>
+        <origin xyz="0 0 0" rpy="0 0 0"/>
+        <mass value="${suspension_mass}"/>
+        <!-- Compact hub / suspension carrier approximation. -->
+        <inertia
+          ixx="0.001" ixy="0.0" ixz="0.0"
+          iyy="0.001" iyz="0.0" izz="0.001"/>
+      </inertial>
+    </link>
+    <joint name="${prefix}_suspension_joint" type="prismatic">
+      <parent link="base_link"/>
+      <child link="${prefix}_suspension_link"/>
+      <origin xyz="${x} ${y} ${wheel_center_z}" rpy="0 0 0"/>
+      <axis xyz="0 0 1"/>
+      <limit
+        lower="${suspension_lower_limit}"
+        upper="${suspension_upper_limit}"
+        effort="5000.0" velocity="2.0"/>
+      <dynamics damping="${suspension_damping}" friction="0.0"/>
+    </joint>
+    <!-- These Gazebo extensions become SDF joint-axis spring dynamics. -->
+    <gazebo reference="${prefix}_suspension_joint">
+      <springReference>${suspension_reference}</springReference>
+      <springStiffness>${suspension_stiffness}</springStiffness>
+    </gazebo>
     <link name="${prefix}_wheel_link">
       <inertial>
@@ -72,6 +107,6 @@
       </inertial>
       <!--
-        This primitive is slightly inset into the wheels already present in
-        the full-body DAE, avoiding prominent duplicate wheel visuals.
+        This primitive slightly oversizes the wheels already present in the
+        full-body DAE so the moving black wheel masks the fixed mesh wheel.
       -->
       <visual name="wheel_visual">
@@ -91,7 +126,7 @@
     </link>
     <joint name="${prefix}_wheel_joint" type="continuous">
-      <parent link="base_link"/>
+      <parent link="${prefix}_suspension_link"/>
       <child link="${prefix}_wheel_link"/>
-      <origin xyz="${x} ${y} ${wheel_center_z}" rpy="0 0 0"/>
+      <origin xyz="0 0 0" rpy="0 0 0"/>
       <axis xyz="0 1 0"/>
       <limit effort="800.0" velocity="20.0"/>

Commit message: fix fwmax weight and CoM

File: urdf/fwmax_skid_steer.urdf.xacro (robot description, xacro)
@@ -14,4 +14,19 @@
   <xacro:property name="base_height" value="0.388"/>
   <xacro:property name="wheel_center_z" value="${wheel_radius - base_height}"/>
+  <!--
+    At zero suspension travel, the nominal ground plane is base_footprint z=0.
+    Keep 1 kg in each carrier and wheel, and place the remaining chassis mass
+    so the complete 195.84 kg robot COM is centred 0.255 m above the ground.
+  -->
+  <xacro:property name="total_mass" value="195.84"/>
+  <xacro:property name="target_com_height" value="0.255"/>
+  <xacro:property name="suspension_mass" value="1.0"/>
+  <xacro:property name="wheel_mass" value="1.0"/>
+  <xacro:property
+    name="base_mass"
+    value="${total_mass - 4.0 * (suspension_mass + wheel_mass)}"/>
+  <xacro:property
+    name="base_com_z"
+    value="${(total_mass * (target_com_height - base_height) - 4.0 * (suspension_mass + wheel_mass) * wheel_center_z) / base_mass}"/>
   <!-- Positive joint travel compresses the wheel upward toward the chassis. -->
   <xacro:property name="suspension_lower_limit" value="-0.030"/>
@@ -19,16 +34,16 @@
   <xacro:property name="suspension_stiffness" value="20000.0"/>
   <xacro:property name="suspension_damping" value="925.0"/>
-  <!-- Preload supports the 117 kg sprung chassis at zero joint travel. -->
-  <xacro:property name="suspension_reference" value="-0.0143471"/>
+  <!-- Preload supports the sprung chassis at zero joint travel. -->
+  <xacro:property
+    name="suspension_reference"
+    value="${-(base_mass * 9.81 / 4.0) / suspension_stiffness}"/>
+  <xacro:property
+    name="nominal_wheel_normal_force"
+    value="${total_mass * 9.81 / 4.0}"/>
   <!--
-    Total mass is 125 kg: 117 kg for the chassis, plus a 1 kg suspension
-    carrier and a 1 kg wheel at each corner. The chassis inertial offset makes
-    the assembled robot's centre of mass coincide with the base_link origin at
-    the designed loaded equilibrium position (zero joint travel).
+    Total mass is 195.84 kg: 187.84 kg for the chassis, plus a 1 kg suspension
+    carrier and a 1 kg wheel at each corner. At the designed loaded equilibrium
+    position, the assembled COM is at x=0, y=0, z=-0.133 m in base_link.
   -->
-  <xacro:property name="base_mass" value="117.0"/>
-  <xacro:property name="base_com_z" value="0.017982905983"/>
-  <xacro:property name="suspension_mass" value="1.0"/>
-  <xacro:property name="wheel_mass" value="1.0"/>
   <material name="fwmax_body_dark_silver">
     <color rgba="0.32 0.34 0.37 1.0"/>
@@ -45,6 +60,9 @@
       <!-- Box approximation based on the 0.96 x 0.55 x 0.395 m envelope. -->
       <inertia
-        ixx="4.470618750" ixy="0.0" ixz="0.0"
-        iyy="10.506843750" iyz="0.0" izz="11.934975000"/>
+        ixx="${base_mass / 12.0 * (0.55 * 0.55 + 0.395 * 0.395)}"
+        ixy="0.0" ixz="0.0"
+        iyy="${base_mass / 12.0 * (0.96 * 0.96 + 0.395 * 0.395)}"
+        iyz="0.0"
+        izz="${base_mass / 12.0 * (0.96 * 0.96 + 0.55 * 0.55)}"/>
     </inertial>
     <visual name="fwmax_dae_visual">
@@ -58,8 +76,14 @@
     </visual>
     <!-- Keep the expensive detailed DAE out of the contact calculation. -->
-    <collision name="base_collision">
+    <!-- <collision name="base_collision">
       <origin xyz="0 0 -0.158" rpy="0 0 0"/>
       <geometry>
         <box size="0.76 0.40 0.22"/>
+      </geometry>
+    </collision> -->
+    <collision name="base_collision">
+      <origin xyz="0 0 0.032" rpy="0 0 0"/>
+      <geometry>
+        <box size="0.76 0.40 0.60"/>
       </geometry>
     </collision>
@@ -177,5 +201,5 @@
         <slip_compliance_lateral>0.2</slip_compliance_lateral>
         <slip_compliance_longitudinal>0.1</slip_compliance_longitudinal>
-        <wheel_normal_force>306.6</wheel_normal_force>
+        <wheel_normal_force>${nominal_wheel_normal_force}</wheel_normal_force>
         <wheel_radius>${wheel_radius}</wheel_radius>
       </wheel>
@@ -183,5 +207,5 @@
         <slip_compliance_lateral>0.2</slip_compliance_lateral>
         <slip_compliance_longitudinal>0.1</slip_compliance_longitudinal>
-        <wheel_normal_force>306.6</wheel_normal_force>
+        <wheel_normal_force>${nominal_wheel_normal_force}</wheel_normal_force>
         <wheel_radius>${wheel_radius}</wheel_radius>
       </wheel>
@@ -189,5 +213,5 @@
         <slip_compliance_lateral>0.2</slip_compliance_lateral>
         <slip_compliance_longitudinal>0.1</slip_compliance_longitudinal>
-        <wheel_normal_force>306.6</wheel_normal_force>
+        <wheel_normal_force>${nominal_wheel_normal_force}</wheel_normal_force>
         <wheel_radius>${wheel_radius}</wheel_radius>
       </wheel>
@@ -195,5 +219,5 @@
         <slip_compliance_lateral>0.2</slip_compliance_lateral>
         <slip_compliance_longitudinal>0.1</slip_compliance_longitudinal>
-        <wheel_normal_force>306.6</wheel_normal_force>
+        <wheel_normal_force>${nominal_wheel_normal_force}</wheel_normal_force>
         <wheel_radius>${wheel_radius}</wheel_radius>
       </wheel>

Commit message: change wheels mass

File: urdf/fwmax_skid_steer.urdf.xacro (robot description, xacro)
@@ -22,5 +22,5 @@
   <xacro:property name="target_com_height" value="0.255"/>
   <xacro:property name="suspension_mass" value="1.0"/>
-  <xacro:property name="wheel_mass" value="1.0"/>
+  <xacro:property name="wheel_mass" value="5.0"/>
   <xacro:property
     name="base_mass"

Commit message: add fwmax sensor config

File: urdf/fwmax_skid_steer.urdf.xacro (robot description, xacro)
@@ -6,4 +6,10 @@
     primitives are used for collision and wheel contact.
   -->
+  <xacro:arg name="namespace" default=""/>
+  <xacro:arg name="is_sim" default="true"/>
+  <xacro:include
+    filename="$(find clearpath_sensors_description)/urdf/ouster_os1.urdf.xacro"/>
+  <xacro:include
+    filename="$(find clearpath_sensors_description)/urdf/intel_realsense.urdf.xacro"/>
   <xacro:property name="wheel_radius" value="0.125"/>
   <xacro:property name="wheel_width" value="0.080"/>
@@ -83,7 +89,7 @@
     </collision> -->
     <collision name="base_collision">
-      <origin xyz="0 0 0.032" rpy="0 0 0"/>
+      <origin xyz="0 0 0.10" rpy="0 0 0"/>
       <geometry>
-        <box size="0.76 0.40 0.60"/>
+        <box size="0.76 0.40 0.80"/>
       </geometry>
     </collision>
@@ -94,4 +100,49 @@
     <origin xyz="0 0 ${base_height}" rpy="0 0 0"/>
   </joint>
+  <!--
+    Ouster OS1-64. The imported model places its measurement frame 0.060695 m
+    above the mounting origin (base height 0.0225 m + sensor offset 0.038195 m).
+    Offset the mount so the requested os_sensor frame is exactly at
+    xyz="0.32 0.0 0.505" relative to base_link.
+  -->
+  <xacro:ouster_os1
+    name="os1_64"
+    parent_link="base_link"
+    samples_v="64">
+    <origin
+      xyz="0.32 0.0 0.505"
+      rpy="0.0 0.0 0.0"/>
+  </xacro:ouster_os1>
+  <!-- Alias the imported Ouster measurement frame to the requested name. -->
+  <link name="os_sensor"/>
+  <joint name="os_sensor_joint" type="fixed">
+    <parent link="os1_64_sensor_link"/>
+    <child link="os_sensor"/>
+    <origin xyz="0 0 0" rpy="0 0 0"/>
+  </joint>
+  <!--
+    RealSense D435. Its imported macro defines camera_link 0.0106, 0.0175,
+    0.0125 m from the bottom-screw frame. Compensate that internal offset so
+    base_link -> camera_link is exactly xyz="0.41 0.01 0.335" and
+    rpy="0.0 0.7854 0.0".
+  -->
+  <xacro:property name="camera_pitch" value="0.7854"/>
+  <xacro:property name="camera_internal_x" value="0.0106"/>
+  <xacro:property name="camera_internal_y" value="0.0175"/>
+  <xacro:property name="camera_internal_z" value="0.0125"/>
+  <xacro:property
+    name="camera_mount_x"
+    value="${0.41 - (cos(camera_pitch) * camera_internal_x + sin(camera_pitch) * camera_internal_z)}"/>
+  <xacro:property
+    name="camera_mount_y"
+    value="${0.01 - camera_internal_y}"/>
+  <xacro:property
+    name="camera_mount_z"
+    value="${0.335 - (-sin(camera_pitch) * camera_internal_x + cos(camera_pitch) * camera_internal_z)}"/>
+  <xacro:intel_realsense name="camera" parent_link="base_link">
+    <origin
+      xyz="${camera_mount_x} ${camera_mount_y} ${camera_mount_z}"
+      rpy="0.0 ${camera_pitch} 0.0"/>
+  </xacro:intel_realsense>
   <xacro:macro name="fwmax_wheel" params="prefix x y">
     <link name="${prefix}_suspension_link">
